File: docs/wiring/mini_vending_machine/gantry_node.kicad_sch (KiCad schematic)
At the start: 5 parts, among them M1 Stepper_Motor_bipolar, M2 Stepper_Motor_bipolar, U1 STM32 Blackpill F411CEU6, U2 TMC2209-LA, U3 TMC2209-LA

Commit message: schematics: gantry, power, can bus
Parts:
- removed M1: Stepper_Motor_bipolar, Package_DFN_QFN:VQFN-28-1EP_5x5mm_P0.5mm_EP3.7x3.7mm_ThermalVias, symbol Motor:Stepper_Motor_bipolar
- removed M2: Stepper_Motor_bipolar, symbol Motor:Stepper_Motor_bipolar
- removed U2, U3: TMC2209-LA, Package_DFN_QFN:VQFN-28-1EP_5x5mm_P0.5mm_EP3.7x3.7mm_ThermalVias, symbol Driver_Motor:TMC2209-LA
- added C1, C2: 100nF, symbol Device:C_US
- added R1, R2: 10k, symbol Device:R_US
Connections:
- net GND: now also U1.31 (A10), C1.2, C2.2, R1.2, R2.2
- net SPI CLK: now reaches U1.15 (A5)
- net at U1.16 (A6): no longer names the net of U1.16 (A6)
- net SPI MOSI: now reaches U1.17 (A7)
- net SPI CAN CS: now reaches U1.18 (B0)
- net CAN Interrupt: now reaches U1.19 (B1)
- net CAN +VLOGIC: now reaches U1.24 (3V3)
- net Y_Limit_Signal: now reaches U1.25 (B12)
- net Y_Limit_Signal: now also C1.1, R1.1
- net X_Limit_Signal: now reaches U1.27 (B14)
- net X_Limit_Signal: now also C2.1, R2.1
- net Shared Steppers UART: now reaches U1.30 (A9)
- net Y_DIR: now reaches U1.39 (B3)
- net Y_STEP: now reaches U1.40 (B4)
- net Y_EN: now reaches U1.41 (B5)
- net X_DIR: now reaches U1.43 (B7)
- net X_STEP: now reaches U1.45 (B8)
- net X_EN: now reaches U1.46 (B9)
- net Step +VLOGIC: now reaches U1.48 (3V3)
- no-connect marks 0 -> 18
Other:
- added sheet Modified MCP2515 CAN Module (modified_mcp2515_can_module.kicad_sch)
- added sheet Stepper Module X (stepper_module.kicad_sch)
- added sheet Stepper Module Y (stepper_module.kicad_sch)
- note added: "Gantry Node"
- company: (none) -> AO Embedded
- title: (none) -> Gantry Node
- moved on the sheet: U1
