File: docs/wiring/mini_vending_machine/mini_vending_machine.kicad_sch (KiCad schematic)
At the start: 0 parts

Commit message: schematics: gantry, power, can bus
Parts:
- added J13, J14, J15: Node Conn, symbol Connector:Conn_01x02_Pin
- added R5, R6: 120R, symbol Device:R_US
Connections:
- new net CANH: J13.1 (Pin_1), J14.2 (Pin_2), J15.1 (Pin_1), R5.1, R6.1
- new net CANL: J13.2 (Pin_2), J14.1 (Pin_1), J15.2 (Pin_2), R5.2, R6.2
Other:
- added sheet Power Module (power_module.kicad_sch)
- sheet Gantry Node ports: added CANH, CANL; removed +5V, GND
- note added: "CAN Bus"
- note added: "Mini Vending Machine"
